File: hardware/CH340USBC/CH340USBC.kicad_pcb (KiCad board)
At the start: 2 copper layers, 1 part, among them U1 CH340E

Commit message: feat: update schematic
Parts:
- added J1: Qwiic_RA, PCM_SparkFun-Connector:JST_1x04_P1.0mm_Horizontal_SMD, F.Cu at (120.1, 73.8)
- added J2: USB_C_Receptacle_USB2.0_16P, Connector_USB:USB_C_Receptacle_Palconn_UTC16-G, F.Cu at (116.8, 107.6)
