File: hardware/CH340USBC/CH340USBC.kicad_sch (KiCad schematic)
At the start: 1 part, among them U1 CH340E

Commit message: feat: update schematic
Parts:
- added J1: Qwiic_RA, PCM_SparkFun-Connector:JST_1x04_P1.0mm_Horizontal_SMD, symbol PCM_SparkFun-Connector:Qwiic_Horizontal
- added J2: USB_C_Receptacle_USB2.0_16P, Connector_USB:USB_C_Receptacle_Palconn_UTC16-G, symbol Connector:USB_C_Receptacle_USB2.0_16P
Connections:
- new net: J2.A1 (GND), J2.A12 (GND), J2.B1 (GND), J2.B12 (GND)
- new net: J2.A4 (VBUS), J2.A9 (VBUS), J2.B4 (VBUS), J2.B9 (VBUS)
